File: Sweep High/Switch Plate/sweep-high_plate.kicad_pcb (KiCad board)
At the start: 2 copper layers, 112.1 x 95.2 mm, 22 parts, among them SW10 SW_Push, SW11 SW_Push, SW12 SW_Push, SW14 SW_Push, SW15 SW_Push, SW16 SW_Push, SW17 SW_Push, SW18 SW_Push, SW2 SW_Push, SW20 SW_Push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

Commit message: lots of worky
Parts:
- removed ?: , 
- H2, H5, H6, H8: footprint MountingHole:MountingHole_3.7mm -> MountingHole:MountingHole_2.2mm_M2
- moved H8 8.88 mm to (55.6, 121.6)
- moved H6 7.90 mm to (99.4, 127.7)
- moved H5 2.38 mm to (53.4, 66.7)
- moved H2 1.94 mm to (112.1, 56.6)
Changed lines of the file:
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@@
     (fp_line (start 7 7) (end 7 -7) (layer "Edge.Cuts") (width 0.15))
   )
-  (footprint "MountingHole:MountingHole_3.7mm" (layer "F.Cu")
-    (at 62.052 115.502)
-    (descr "Mounting Hole 3.7mm, no annular")
-    (tags "mounting hole 3.7mm no annular")
+  (footprint "MountingHole:MountingHole_2.2mm_M2" (layer "F.Cu")
+    (at 55.6 121.6)
+    (descr "Mounting Hole 2.2mm, no annular, M2")
+    (tags "mounting hole 2.2mm no annular m2")
     (property "Sheetfile" "sweepv2.kicad_sch")
     (property "Sheetname" "")
-    (attr exclude_from_pos_files)
-    (fp_text reference "H8" (at 0 -4.7) (layer "F.SilkS")
+    (attr exclude_from_pos_files exclude_from_bom)
+    (fp_text reference "H8" (at 0 -3.2) (layer "F.SilkS")
       (effects (font (size 1 1) (thickness 0.15)))
     )
-    (fp_text value "MountingHole" (at 0 4.7) (layer "F.Fab")
+    (fp_text value "MountingHole" (at 0 3.2) (layer "F.Fab")
       (effects (font (size 1 1) (thickness 0.15)))
     )
@@
       (effects (font (size 1 1) (thickness 0.15)))
     )
-    (fp_circle (center 0 0) (end 3.7 0) (layer "Cmts.User") (width 0.15) (fill none))
-    (fp_circle (center 0 0) (end 3.95 0) (layer "F.CrtYd") (width 0.05) (fill none))
-    (pad "" np_thru_hole circle (at 0 0) (size 3.7 3.7) (drill 3.7) (layers F&B.Cu *.Mask))
+    (fp_circle (center 0 0) (end 2.2 0) (layer "Cmts.User") (width 0.15) (fill none))
+    (fp_circle (center 0 0) (end 2.45 0) (layer "F.CrtYd") (width 0.05) (fill none))
+    (pad "" np_thru_hole circle (at 0 0) (size 2.2 2.2) (drill 2.2) (layers *.Cu *.Mask))
   )
-  (footprint "" (layer "F.Cu")
-    (at 62.052 115.502)
-    (fp_text reference "" (at 0 0) (layer "F.SilkS")
-      (effects (font (size 1.27 1.27) (thickness 0.15)))
-    )
-    (fp_text value "" (at 0 0) (layer "F.SilkS")
-      (effects (font (size 1.27 1.27) (thickness 0.15)))
-    )
-    (pad "" np_thru_hole circle (at 0 0) (size 3.7 3.7) (drill 3.7) (layers F&B.Cu *.Mask))
-  )
-  (footprint "MountingHole:MountingHole_3.7mm" (layer "F.Cu")
-    (at 54.178 64.448)
-    (descr "Mounting Hole 3.7mm, no annular")
-    (tags "mounting hole 3.7mm no annular")
+  (footprint "MountingHole:MountingHole_2.2mm_M2" (layer "F.Cu")
+    (at 53.4 66.7)
+    (descr "Mounting Hole 2.2mm, no annular, M2")
+    (tags "mounting hole 2.2mm no annular m2")
     (property "Sheetfile" "sweepv2.kicad_sch")
     (property "Sheetname" "")
-    (attr exclude_from_pos_files)
-    (fp_text reference "H5" (at 0 -4.7) (layer "F.SilkS")
+    (attr exclude_from_pos_files exclude_from_bom)
+    (fp_text reference "H5" (at 0 -3.2) (layer "F.SilkS")
       (effects (font (size 1 1) (thickness 0.15)))
     )
-    (fp_text value "MountingHole" (at 0 4.7) (layer "F.Fab")
+    (fp_text value "MountingHole" (at 0 3.2) (layer "F.Fab")
       (effects (font (size 1 1) (thickness 0.15)))
     )
@@
       (effects (font (size 1 1) (thickness 0.15)))
     )
-    (fp_circle (center 0 0) (end 3.7 0) (layer "Cmts.User") (width 0.15) (fill none))
-    (fp_circle (center 0 0) (end 3.95 0) (layer "F.CrtYd") (width 0.05) (fill none))
-    (pad "" np_thru_hole circle (at 0 0) (size 3.7 3.7) (drill 3.7) (layers F&B.Cu *.Mask))
+    (fp_circle (center 0 0) (end 2.2 0) (layer "Cmts.User") (width 0.15) (fill none))
+    (fp_circle (center 0 0) (end 2.45 0) (layer "F.CrtYd") (width 0.05) (fill none))
+    (pad "" np_thru_hole circle (at 0 0) (size 2.2 2.2) (drill 2.2) (layers *.Cu *.Mask))
   )
-  (footprint "MountingHole:MountingHole_3.7mm" (layer "F.Cu")
-    (at 98.882 119.82)
-    (descr "Mounting Hole 3.7mm, no annular")
-    (tags "mounting hole 3.7mm no annular")
+  (footprint "MountingHole:MountingHole_2.2mm_M2" (layer "F.Cu")
+    (at 99.4 127.7)
+    (descr "Mounting Hole 2.2mm, no annular, M2")
+    (tags "mounting hole 2.2mm no annular m2")
     (property "Sheetfile" "sweepv2.kicad_sch")
     (property "Sheetname" "")
-    (attr exclude_from_pos_files)
-    (fp_text reference "H6" (at 0 -4.7) (layer "F.SilkS")
+    (attr exclude_from_pos_files exclude_from_bom)
+    (fp_text reference "H6" (at 0 -3.2) (layer "F.SilkS")
       (effects (font (size 1 1) (thickness 0.15)))
     )
-    (fp_text value "MountingHole" (at 6.388 -34.29) (layer "F.Fab")
+    (fp_text value "MountingHole" (at 0 3.2) (layer "F.Fab")
       (effects (font (size 1 1) (thickness 0.15)))
     )
@@
       (effects (font (size 1 1) (thickness 0.15)))
     )
-    (fp_circle (center 0 0) (end 3.7 0) (layer "Cmts.User") (width 0.15) (fill none))
-    (fp_circle (center 0 0) (end 3.95 0) (layer "F.CrtYd") (width 0.05) (fill none))
-    (pad "" np_thru_hole circle (at 0 0) (size 3.7 3.7) (drill 3.7) (layers F&B.Cu *.Mask))
+    (fp_circle (center 0 0) (end 2.2 0) (layer "Cmts.User") (width 0.15) (fill none))
+    (fp_circle (center 0 0) (end 2.45 0) (layer "F.CrtYd") (width 0.05) (fill none))
+    (pad "" np_thru_hole circle (at 0 0) (size 2.2 2.2) (drill 2.2) (layers *.Cu *.Mask))
   )
-  (footprint "MountingHole:MountingHole_3.7mm" (layer "F.Cu")
-    (at 113.868 55.812)
-    (descr "Mounting Hole 3.7mm, no annular")
-    (tags "mounting hole 3.7mm no annular")
+  (footprint "MountingHole:MountingHole_2.2mm_M2" (layer "F.Cu")
+    (at 112.1 56.6)
+    (descr "Mounting Hole 2.2mm, no annular, M2")
+    (tags "mounting hole 2.2mm no annular m2")
     (property "Sheetfile" "sweepv2.kicad_sch")
     (property "Sheetname" "")
-    (attr exclude_from_pos_files)
-    (fp_text reference "H2" (at 0 -4.7) (layer "F.SilkS")
+    (attr exclude_from_pos_files exclude_from_bom)
+    (fp_text reference "H2" (at 0 -3.2) (layer "F.SilkS")
       (effects (font (size 1 1) (thickness 0.15)))
     )
-    (fp_text value "MountingHole" (at 0 4.7) (layer "F.Fab")
+    (fp_text value "MountingHole" (at 0 3.2) (layer "F.Fab")
       (effects (font (size 1 1) (thickness 0.15)))
     )
@@
       (effects (font (size 1 1) (thickness 0.15)))
     )
-    (fp_circle (center 0 0) (end 3.7 0) (layer "Cmts.User") (width 0.15) (fill none))
-    (fp_circle (center 0 0) (end 3.95 0) (layer "F.CrtYd") (width 0.05) (fill none))
-    (pad "" np_thru_hole circle (at 0 0) (size 3.7 3.7) (drill 3.7) (layers F&B.Cu *.Mask))
+    (fp_circle (center 0 0) (end 2.2 0) (layer "Cmts.User") (width 0.15) (fill none))
+    (fp_circle (center 0 0) (end 2.45 0) (layer "F.CrtYd") (width 0.05) (fill none))
+    (pad "" np_thru_hole circle (at 0 0) (size 2.2 2.2) (drill 2.2) (layers *.Cu *.Mask))
   )
   (gr_line (start 147.161679 123.613657) (end 135.71 143.699265) (layer "Edge.Cuts") (width 0.05))
