File: Sweep High/MainPCB/sweep-high.kicad_sch (KiCad schematic)
At the start: 54 parts, among them J1 AudioJack4dpb, J2 AudioJack4dpb, SW10 SW_Push, SW10_r1 SW_Push, SW11 SW_Push, SW11_r1 SW_Push, SW12 SW_Push, SW12_r1 SW_Push, SW13_r1 SW_Push, SW14 SW_Push, SW14_r1 SW_Push, SW15 SW_Push, SW15_r1 SW_Push, SW16 SW_Push, SW16_r1 SW_Push, SW17 SW_Push, SW17_r1 SW_Push, SW18 SW_Push, SW18_r1 SW_Push, SW2 SW_Push, SW20 SW_Push, SW21 SW_Push, SW2_r1 SW_Push, SW3 SW_Push, SW3_r1 SW_Push, SW4 SW_Push, SW4_r1 SW_Push, SW5 SW_Push, SW5_r1 SW_Push, SW6 SW_Push, SW6_r1 SW_Push, SW7_r1 SW_Push, SW8 SW_Push, SW8_r1 SW_Push, SW9 SW_Push, SW9_r1 SW_Push, U1 ProMicro-kbd, U2 ProMicro-kbd

Commit message: more missed corrections
Parts:
- H5: renamed from H?; footprint (none) -> MountingHole:MountingHole_3.2mm_M3
- gave numbers to parts that had none: 7
Changed lines of the file:
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@@
   (symbol (lib_id "Mechanical:MountingHole") (at 152.4 156.845 0) (unit 1)
     (in_bom yes) (on_board yes) (fields_autoplaced)
-    (property "Reference" "H?" (id 0) (at 154.94 155.5749 0)
+    (property "Reference" "H2" (id 0) (at 154.94 155.5749 0)
       (effects (font (size 1.27 1.27)) (justify left))
     )
@@
   (symbol (lib_id "Mechanical:MountingHole") (at 153.67 82.55 0) (unit 1)
     (in_bom yes) (on_board yes) (fields_autoplaced)
-    (property "Reference" "H?" (id 0) (at 156.21 81.2799 0)
+    (property "Reference" "H6" (id 0) (at 156.21 81.2799 0)
       (effects (font (size 1.27 1.27)) (justify left))
     )
@@
   (symbol (lib_id "Mechanical:MountingHole") (at 153.67 86.995 0) (unit 1)
     (in_bom yes) (on_board yes) (fields_autoplaced)
-    (property "Reference" "H?" (id 0) (at 156.21 85.7249 0)
+    (property "Reference" "H7" (id 0) (at 156.21 85.7249 0)
       (effects (font (size 1.27 1.27)) (justify left))
     )
@@
   (symbol (lib_id "Mechanical:MountingHole") (at 153.67 78.105 0) (unit 1)
     (in_bom yes) (on_board yes) (fields_autoplaced)
-    (property "Reference" "H?" (id 0) (at 156.21 76.8349 0)
+    (property "Reference" "H5" (id 0) (at 156.21 76.8349 0)
       (effects (font (size 1.27 1.27)) (justify left))
     )
@@
       (effects (font (size 1.27 1.27)) (justify left))
     )
-    (property "Footprint" "" (id 2) (at 153.67 78.105 0)
+    (property "Footprint" "MountingHole:MountingHole_3.2mm_M3" (id 2) (at 153.67 78.105 0)
       (effects (font (size 1.27 1.27)) hide)
     )
@@
   (symbol (lib_id "Mechanical:MountingHole") (at 152.4 152.4 0) (unit 1)
     (in_bom yes) (on_board yes) (fields_autoplaced)
-    (property "Reference" "H?" (id 0) (at 154.94 151.1299 0)
+    (property "Reference" "H1" (id 0) (at 154.94 151.1299 0)
       (effects (font (size 1.27 1.27)) (justify left))
     )
@@
   (symbol (lib_id "Mechanical:MountingHole") (at 152.4 161.29 0) (unit 1)
     (in_bom yes) (on_board yes) (fields_autoplaced)
-    (property "Reference" "H?" (id 0) (at 154.94 160.0199 0)
+    (property "Reference" "H3" (id 0) (at 154.94 160.0199 0)
       (effects (font (size 1.27 1.27)) (justify left))
     )
@@
   (symbol (lib_id "Mechanical:MountingHole") (at 153.67 91.44 0) (unit 1)
     (in_bom yes) (on_board yes) (fields_autoplaced)
-    (property "Reference" "H?" (id 0) (at 156.21 90.1699 0)
+    (property "Reference" "H8" (id 0) (at 156.21 90.1699 0)
       (effects (font (size 1.27 1.27)) (justify left))
     )
@@
   (symbol (lib_id "Mechanical:MountingHole") (at 152.4 165.735 0) (unit 1)
     (in_bom yes) (on_board yes) (fields_autoplaced)
-    (property "Reference" "H?" (id 0) (at 154.94 164.4649 0)
+    (property "Reference" "H4" (id 0) (at 154.94 164.4649 0)
       (effects (font (size 1.27 1.27)) (justify left))
     )
@@
       (reference "BatGND4") (unit 1) (value "MountingHole_Pad") (footprint "Connector_Pin:Pin_D1.4mm_L8.5mm_W2.8mm_FlatFork")
     )
+    (path "/a6d5e28c-e4f9-48de-98d4-4a7c6786c0db"
+      (reference "H1") (unit 1) (value "MountingHole") (footprint "MountingHole:MountingHole_3.2mm_M3")
+    )
     (path "/32046e7d-db36-4244-a11b-27c70ad03618"
-      (reference "H?") (unit 1) (value "MountingHole") (footprint "MountingHole:MountingHole_3.2mm_M3")
+      (reference "H2") (unit 1) (value "MountingHole") (footprint "MountingHole:MountingHole_3.2mm_M3")
+    )
+    (path "/b0db1011-cfc4-44e4-b449-76f6d8240296"
+      (reference "H3") (unit 1) (value "MountingHole") (footprint "MountingHole:MountingHole_3.2mm_M3")
+    )
+    (path "/e1960dc1-7cde-446b-9532-8464ccedbaba"
+      (reference "H4") (unit 1) (value "MountingHole") (footprint "MountingHole:MountingHole_3.2mm_M3")
+    )
+    (path "/8affb2b3-e3ad-4e1c-a2fe-16a165cbf33a"
+      (reference "H5") (unit 1) (value "MountingHole") (footprint "MountingHole:MountingHole_3.2mm_M3")
     )
     (path "/6f449a0c-65d3-4351-8814-f85236fe36a7"
-      (reference "H?") (unit 1) (value "MountingHole") (footprint "MountingHole:MountingHole_3.2mm_M3")
+      (reference "H6") (unit 1) (value "MountingHole") (footprint "MountingHole:MountingHole_3.2mm_M3")
     )
     (path "/8ad589ef-ed7c-4c96-89a5-ba65952bdb30"
-      (reference "H?") (unit 1) (value "MountingHole") (footprint "MountingHole:MountingHole_3.2mm_M3")
-    )
-    (path "/8affb2b3-e3ad-4e1c-a2fe-16a165cbf33a"
-      (reference "H?") (unit 1) (value "MountingHole") (footprint "MountingHole:MountingHole_3.2mm_M3")
-    )
-    (path "/a6d5e28c-e4f9-48de-98d4-4a7c6786c0db"
-      (reference "H?") (unit 1) (value "MountingHole") (footprint "MountingHole:MountingHole_3.2mm_M3")
-    )
-    (path "/b0db1011-cfc4-44e4-b449-76f6d8240296"
-      (reference "H?") (unit 1) (value "MountingHole") (footprint "MountingHole:MountingHole_3.2mm_M3")
+      (reference "H7") (unit 1) (value "MountingHole") (footprint "MountingHole:MountingHole_3.2mm_M3")
     )
     (path "/d93bd2ed-9a20-4726-9076-8c57f7589a70"
-      (reference "H?") (unit 1) (value "MountingHole") (footprint "MountingHole:MountingHole_3.2mm_M3")
-    )
-    (path "/e1960dc1-7cde-446b-9532-8464ccedbaba"
-      (reference "H?") (unit 1) (value "MountingHole") (footprint "MountingHole:MountingHole_3.2mm_M3")
+      (reference "H8") (unit 1) (value "MountingHole") (footprint "MountingHole:MountingHole_3.2mm_M3")
     )
     (path "/00000000-0000-0000-0000-0000605e7e3e"

Commit message: some adjustments and stuff, changed my mind on some footprints and also missed some stuff I used for alignment and checking
Parts:
- J1, J2: footprint Connector_Audio:Jack_3.5mm_PJ320D_Horizontal -> env_extra:PJ-320A
Changed lines of the file:
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@@
     (property "Reference" "J1" (id 0) (at 120.8278 59.055 0))
     (property "Value" "AudioJack4dpb" (id 1) (at 120.8278 61.3664 0))
-    (property "Footprint" "Connector_Audio:Jack_3.5mm_PJ320D_Horizontal" (id 2) (at 121.92 67.31 0)
+    (property "Footprint" "env_extra:PJ-320A" (id 2) (at 121.92 67.31 0)
       (effects (font (size 1.27 1.27)) hide)
     )
@@
     (property "Reference" "J2" (id 0) (at 122.0978 158.115 0))
     (property "Value" "AudioJack4dpb" (id 1) (at 122.0978 160.4264 0))
-    (property "Footprint" "Connector_Audio:Jack_3.5mm_PJ320D_Horizontal" (id 2) (at 123.19 166.37 0)
+    (property "Footprint" "env_extra:PJ-320A" (id 2) (at 123.19 166.37 0)
       (effects (font (size 1.27 1.27)) hide)
     )
@@
     )
     (path "/00000000-0000-0000-0000-0000605e7e3e"
-      (reference "J1") (unit 1) (value "AudioJack4dpb") (footprint "Connector_Audio:Jack_3.5mm_PJ320D_Horizontal")
+      (reference "J1") (unit 1) (value "AudioJack4dpb") (footprint "env_extra:PJ-320A")
     )
     (path "/00000000-0000-0000-0000-0000608f2563"
-      (reference "J2") (unit 1) (value "AudioJack4dpb") (footprint "Connector_Audio:Jack_3.5mm_PJ320D_Horizontal")
+      (reference "J2") (unit 1) (value "AudioJack4dpb") (footprint "env_extra:PJ-320A")
     )
     (path "/00000000-0000-0000-0000-0000604ea4f3"
