File: Sweep v2.2/_MainPCB/sweepv2.kicad_sch (KiCad schematic)
At the start: 54 parts, among them J1 AudioJack4dpb, J2 AudioJack4dpb, SW1 SW_Push, SW10 SW_Push, SW11 SW_Push, SW11_r1 SW_Push, SW12 SW_Push, SW12_r1 SW_Push, SW13_r1 SW_Push, SW14 SW_Push, SW15 SW_Push, SW15_r1 SW_Push, SW16 SW_Push, SW16_r1 SW_Push, SW17 SW_Push, SW17_r1 SW_Push, SW18 SW_Push, SW18_r1 SW_Push, SW2 SW_Push, SW20 SW_Push, SW21 SW_Push, SW2_r1 SW_Push, SW3 SW_Push, SW3_r1 SW_Push, SW4 SW_Push, SW4_r1 SW_Push, SW5 SW_Push, SW5_r1 SW_Push, SW6 SW_Push, SW6_r1 SW_Push, SW7 SW_Push, SW7_r1 SW_Push, SW8 SW_Push, SW8_r1 SW_Push, SW9 SW_Push, SW9_r1 SW_Push, U1 ProMicro-kbd, U2 ProMicro-kbd

Commit message: some adjustments and stuff, changed my mind on some footprints and also missed some stuff I used for alignment and checking
Parts:
- J1, J2: footprint Connector_Audio:Jack_3.5mm_PJ320D_Horizontal -> env_extra:PJ-320A
Changed lines of the file:
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@@
     (property "Reference" "J1" (id 0) (at 120.8278 59.055 0))
     (property "Value" "AudioJack4dpb" (id 1) (at 120.8278 61.3664 0))
-    (property "Footprint" "Connector_Audio:Jack_3.5mm_PJ320D_Horizontal" (id 2) (at 121.92 67.31 0)
+    (property "Footprint" "env_extra:PJ-320A" (id 2) (at 121.92 67.31 0)
       (effects (font (size 1.27 1.27)) hide)
     )
@@
     (property "Reference" "J2" (id 0) (at 122.0978 158.115 0))
     (property "Value" "AudioJack4dpb" (id 1) (at 122.0978 160.4264 0))
-    (property "Footprint" "Connector_Audio:Jack_3.5mm_PJ320D_Horizontal" (id 2) (at 123.19 166.37 0)
+    (property "Footprint" "env_extra:PJ-320A" (id 2) (at 123.19 166.37 0)
       (effects (font (size 1.27 1.27)) hide)
     )
@@
     )
     (path "/00000000-0000-0000-0000-0000605e7e3e"
-      (reference "J1") (unit 1) (value "AudioJack4dpb") (footprint "Connector_Audio:Jack_3.5mm_PJ320D_Horizontal")
+      (reference "J1") (unit 1) (value "AudioJack4dpb") (footprint "env_extra:PJ-320A")
     )
     (path "/00000000-0000-0000-0000-0000608f2563"
-      (reference "J2") (unit 1) (value "AudioJack4dpb") (footprint "Connector_Audio:Jack_3.5mm_PJ320D_Horizontal")
+      (reference "J2") (unit 1) (value "AudioJack4dpb") (footprint "env_extra:PJ-320A")
     )
     (path "/00000000-0000-0000-0000-0000604ea4f3"
