File: Sweep High/Backplate/sweep-high-backplate.kicad_sch (KiCad schematic)
At the start: 8 parts

Commit message: somehow some more things I missed, namely mount hole sizes
Parts:
- H1, H2, H3, H4, H5, H6, H7, H8: footprint MountingHole:MountingHole_3.2mm_M3 -> MountingHole:MountingHole_2.2mm_M2
Changed lines of the file:
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@@
       (effects (font (size 1.27 1.27)) (justify left))
     )
-    (property "Footprint" "MountingHole:MountingHole_3.2mm_M3" (id 2) (at 152.4 156.845 0)
+    (property "Footprint" "MountingHole:MountingHole_2.2mm_M2" (id 2) (at 152.4 156.845 0)
       (effects (font (size 1.27 1.27)) hide)
     )
@@
       (effects (font (size 1.27 1.27)) (justify left))
     )
-    (property "Footprint" "MountingHole:MountingHole_3.2mm_M3" (id 2) (at 153.67 82.55 0)
+    (property "Footprint" "MountingHole:MountingHole_2.2mm_M2" (id 2) (at 153.67 82.55 0)
       (effects (font (size 1.27 1.27)) hide)
     )
@@
       (effects (font (size 1.27 1.27)) (justify left))
     )
-    (property "Footprint" "MountingHole:MountingHole_3.2mm_M3" (id 2) (at 153.67 86.995 0)
+    (property "Footprint" "MountingHole:MountingHole_2.2mm_M2" (id 2) (at 153.67 86.995 0)
       (effects (font (size 1.27 1.27)) hide)
     )
@@
       (effects (font (size 1.27 1.27)) (justify left))
     )
-    (property "Footprint" "MountingHole:MountingHole_3.2mm_M3" (id 2) (at 153.67 78.105 0)
+    (property "Footprint" "MountingHole:MountingHole_2.2mm_M2" (id 2) (at 153.67 78.105 0)
       (effects (font (size 1.27 1.27)) hide)
     )
@@
       (effects (font (size 1.27 1.27)) (justify left))
     )
-    (property "Footprint" "MountingHole:MountingHole_3.2mm_M3" (id 2) (at 152.4 152.4 0)
+    (property "Footprint" "MountingHole:MountingHole_2.2mm_M2" (id 2) (at 152.4 152.4 0)
       (effects (font (size 1.27 1.27)) hide)
     )
@@
       (effects (font (size 1.27 1.27)) (justify left))
     )
-    (property "Footprint" "MountingHole:MountingHole_3.2mm_M3" (id 2) (at 152.4 161.29 0)
+    (property "Footprint" "MountingHole:MountingHole_2.2mm_M2" (id 2) (at 152.4 161.29 0)
       (effects (font (size 1.27 1.27)) hide)
     )
@@
       (effects (font (size 1.27 1.27)) (justify left))
     )
-    (property "Footprint" "MountingHole:MountingHole_3.2mm_M3" (id 2) (at 153.67 91.44 0)
+    (property "Footprint" "MountingHole:MountingHole_2.2mm_M2" (id 2) (at 153.67 91.44 0)
       (effects (font (size 1.27 1.27)) hide)
     )
@@
       (effects (font (size 1.27 1.27)) (justify left))
     )
-    (property "Footprint" "MountingHole:MountingHole_3.2mm_M3" (id 2) (at 152.4 165.735 0)
+    (property "Footprint" "MountingHole:MountingHole_2.2mm_M2" (id 2) (at 152.4 165.735 0)
       (effects (font (size 1.27 1.27)) hide)
     )
@@
   (symbol_instances
     (path "/a6d5e28c-e4f9-48de-98d4-4a7c6786c0db"
-      (reference "H1") (unit 1) (value "MountingHole") (footprint "MountingHole:MountingHole_3.2mm_M3")
+      (reference "H1") (unit 1) (value "MountingHole") (footprint "MountingHole:MountingHole_2.2mm_M2")
     )
     (path "/32046e7d-db36-4244-a11b-27c70ad03618"
-      (reference "H2") (unit 1) (value "MountingHole") (footprint "MountingHole:MountingHole_3.2mm_M3")
+      (reference "H2") (unit 1) (value "MountingHole") (footprint "MountingHole:MountingHole_2.2mm_M2")
     )
     (path "/b0db1011-cfc4-44e4-b449-76f6d8240296"
-      (reference "H3") (unit 1) (value "MountingHole") (footprint "MountingHole:MountingHole_3.2mm_M3")
+      (reference "H3") (unit 1) (value "MountingHole") (footprint "MountingHole:MountingHole_2.2mm_M2")
     )
     (path "/e1960dc1-7cde-446b-9532-8464ccedbaba"
-      (reference "H4") (unit 1) (value "MountingHole") (footprint "MountingHole:MountingHole_3.2mm_M3")
+      (reference "H4") (unit 1) (value "MountingHole") (footprint "MountingHole:MountingHole_2.2mm_M2")
     )
     (path "/8affb2b3-e3ad-4e1c-a2fe-16a165cbf33a"
-      (reference "H5") (unit 1) (value "MountingHole") (footprint "MountingHole:MountingHole_3.2mm_M3")
+      (reference "H5") (unit 1) (value "MountingHole") (footprint "MountingHole:MountingHole_2.2mm_M2")
     )
     (path "/6f449a0c-65d3-4351-8814-f85236fe36a7"
-      (reference "H6") (unit 1) (value "MountingHole") (footprint "MountingHole:MountingHole_3.2mm_M3")
+      (reference "H6") (unit 1) (value "MountingHole") (footprint "MountingHole:MountingHole_2.2mm_M2")
     )
     (path "/8ad589ef-ed7c-4c96-89a5-ba65952bdb30"
-      (reference "H7") (unit 1) (value "MountingHole") (footprint "MountingHole:MountingHole_3.2mm_M3")
+      (reference "H7") (unit 1) (value "MountingHole") (footprint "MountingHole:MountingHole_2.2mm_M2")
     )
     (path "/d93bd2ed-9a20-4726-9076-8c57f7589a70"
-      (reference "H8") (unit 1) (value "MountingHole") (footprint "MountingHole:MountingHole_3.2mm_M3")
+      (reference "H8") (unit 1) (value "MountingHole") (footprint "MountingHole:MountingHole_2.2mm_M2")
     )
   )
