File: Sweep v2.2/_BackPlate/sweepV2_backplate.kicad_pcb (KiCad board)
At the start: 2 copper layers, 216.9 x 86.9 mm, 12 parts

Commit message: somehow some more things I missed, namely mount hole sizes
Other:
- board text added: "Sweep v 2.2 MBUK"
- board text removed: "Face down"
- board text removed: "Sweep v 2.2"
Changed lines of the file:
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@@
     (property "Sheetfile" "sweepV2_backplate.kicad_sch")
     (property "Sheetname" "")
-    (attr exclude_from_pos_files exclude_from_bom)
+    (attr exclude_from_pos_files)
     (fp_text reference "H7" (at 0 -3.2) (layer "F.SilkS")
       (effects (font (size 1 1) (thickness 0.15)))
@@
     (property "Sheetfile" "sweepV2_backplate.kicad_sch")
     (property "Sheetname" "")
-    (attr exclude_from_pos_files exclude_from_bom)
+    (attr exclude_from_pos_files)
     (fp_text reference "H8" (at 0 -3.2) (layer "F.SilkS")
       (effects (font (size 1 1) (thickness 0.15)))
@@
     (property "Sheetfile" "sweepV2_backplate.kicad_sch")
     (property "Sheetname" "")
-    (attr exclude_from_pos_files exclude_from_bom)
+    (attr exclude_from_pos_files)
     (fp_text reference "H5" (at 0 -3.2) (layer "F.SilkS")
       (effects (font (size 1 1) (thickness 0.15)))
@@
     (property "Sheetfile" "sweepV2_backplate.kicad_sch")
     (property "Sheetname" "")
-    (attr exclude_from_pos_files exclude_from_bom)
+    (attr exclude_from_pos_files)
     (fp_text reference "H3" (at 0 -3.2) (layer "F.SilkS")
       (effects (font (size 1 1) (thickness 0.15)))
@@
     (property "Sheetfile" "sweepV2_backplate.kicad_sch")
     (property "Sheetname" "")
-    (attr exclude_from_pos_files exclude_from_bom)
+    (attr exclude_from_pos_files)
     (fp_text reference "H1" (at 0 -3.2) (layer "F.SilkS")
       (effects (font (size 1 1) (thickness 0.15)))
@@
     (property "Sheetfile" "sweepV2_backplate.kicad_sch")
     (property "Sheetname" "")
-    (attr exclude_from_pos_files exclude_from_bom)
+    (attr exclude_from_pos_files)
     (fp_text reference "H6" (at 0 -3.2) (layer "F.SilkS")
       (effects (font (size 1 1) (thickness 0.15)))
@@
     (property "Sheetfile" "sweepV2_backplate.kicad_sch")
     (property "Sheetname" "")
-    (attr exclude_from_pos_files exclude_from_bom)
+    (attr exclude_from_pos_files)
     (fp_text reference "H4" (at 0 -3.2) (layer "F.SilkS")
       (effects (font (size 1 1) (thickness 0.15)))
@@
     (property "Sheetfile" "sweepV2_backplate.kicad_sch")
     (property "Sheetname" "")
-    (attr exclude_from_pos_files exclude_from_bom)
+    (attr exclude_from_pos_files)
     (fp_text reference "H2" (at 0 -3.2) (layer "F.SilkS")
       (effects (font (size 1 1) (thickness 0.15)))
@@
   (gr_line (start 131.5085 77.724) (end 131.2545 77.724) (layer "Edge.Cuts") (width 0.05))
   (gr_arc (start 129.349501 53.848) (mid 130.302 53.203127) (end 131.254499 53.848001) (layer "Edge.Cuts") (width 0.05))
-  (gr_text "Sweep v 2.2" (at 140.97 39.116) (layer "B.SilkS")
-    (effects (font (size 1.5 1.5) (thickness 0.3)) (justify mirror))
+  (gr_text "Sweep v 2.2\nMBUK" (at 146.6 43) (layer "B.SilkS")
+    (effects (font (size 1.5 1.5) (thickness 0.3)) (justify left mirror))
   )
   (gr_text "Sweep is based on the Ferris." (at 166.37 81.788) (layer "B.SilkS")
     (effects (font (size 1.5 1.5) (thickness 0.3)) (justify mirror))
   )
-  (gr_text "Face down" (at 230.378 67.056 90) (layer "F.SilkS")
-    (effects (font (size 1.5 1.5) (thickness 0.3)))
-  )
-  (gr_text "Face down" (at 29.718 66.548 90) (layer "F.SilkS")
-    (effects (font (size 1.5 1.5) (thickness 0.3)))
-  )
   (zone (net 0) (net_name "") (layer "F.Cu") (hatch edge 0.508)
