File: Sweep v2.2/_BackPlate/sweepV2_backplate.kicad_sch (KiCad schematic)
At the start: 8 parts

Commit message: somehow some more things I missed, namely mount hole sizes
Parts:
- H1, H2, H3, H4, H5, H6, H7, H8: footprint MountingHole:MountingHole_3.7mm -> MountingHole:MountingHole_2.2mm_M2
Changed lines of the file:
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@@
       (effects (font (size 1.27 1.27)) (justify left))
     )
-    (property "Footprint" "MountingHole:MountingHole_3.7mm" (id 2) (at 153.67 95.25 0)
+    (property "Footprint" "MountingHole:MountingHole_2.2mm_M2" (id 2) (at 153.67 95.25 0)
       (effects (font (size 1.27 1.27)) hide)
     )
@@
       (effects (font (size 1.27 1.27)) (justify left))
     )
-    (property "Footprint" "MountingHole:MountingHole_3.7mm" (id 2) (at 153.67 90.17 0)
+    (property "Footprint" "MountingHole:MountingHole_2.2mm_M2" (id 2) (at 153.67 90.17 0)
       (effects (font (size 1.27 1.27)) hide)
     )
@@
       (effects (font (size 1.27 1.27)) (justify left))
     )
-    (property "Footprint" "MountingHole:MountingHole_3.7mm" (id 2) (at 134.62 80.01 0)
+    (property "Footprint" "MountingHole:MountingHole_2.2mm_M2" (id 2) (at 134.62 80.01 0)
       (effects (font (size 1.27 1.27)) hide)
     )
@@
       (effects (font (size 1.27 1.27)) (justify left))
     )
-    (property "Footprint" "MountingHole:MountingHole_3.7mm" (id 2) (at 134.62 90.17 0)
+    (property "Footprint" "MountingHole:MountingHole_2.2mm_M2" (id 2) (at 134.62 90.17 0)
       (effects (font (size 1.27 1.27)) hide)
     )
@@
       (effects (font (size 1.27 1.27)) (justify left))
     )
-    (property "Footprint" "MountingHole:MountingHole_3.7mm" (id 2) (at 153.67 80.01 0)
+    (property "Footprint" "MountingHole:MountingHole_2.2mm_M2" (id 2) (at 153.67 80.01 0)
       (effects (font (size 1.27 1.27)) hide)
     )
@@
       (effects (font (size 1.27 1.27)) (justify left))
     )
-    (property "Footprint" "MountingHole:MountingHole_3.7mm" (id 2) (at 134.62 95.25 0)
+    (property "Footprint" "MountingHole:MountingHole_2.2mm_M2" (id 2) (at 134.62 95.25 0)
       (effects (font (size 1.27 1.27)) hide)
     )
@@
       (effects (font (size 1.27 1.27)) (justify left))
     )
-    (property "Footprint" "MountingHole:MountingHole_3.7mm" (id 2) (at 153.67 85.09 0)
+    (property "Footprint" "MountingHole:MountingHole_2.2mm_M2" (id 2) (at 153.67 85.09 0)
       (effects (font (size 1.27 1.27)) hide)
     )
@@
       (effects (font (size 1.27 1.27)) (justify left))
     )
-    (property "Footprint" "MountingHole:MountingHole_3.7mm" (id 2) (at 134.62 85.09 0)
+    (property "Footprint" "MountingHole:MountingHole_2.2mm_M2" (id 2) (at 134.62 85.09 0)
       (effects (font (size 1.27 1.27)) hide)
     )
@@
   (symbol_instances
     (path "/48b659b1-0d3a-4754-8412-bd48e78651ed"
-      (reference "H1") (unit 1) (value "MountingHole") (footprint "MountingHole:MountingHole_3.7mm")
+      (reference "H1") (unit 1) (value "MountingHole") (footprint "MountingHole:MountingHole_2.2mm_M2")
     )
     (path "/eaaa73b7-a6fc-43e9-a08d-428f9d579671"
-      (reference "H2") (unit 1) (value "MountingHole") (footprint "MountingHole:MountingHole_3.7mm")
+      (reference "H2") (unit 1) (value "MountingHole") (footprint "MountingHole:MountingHole_2.2mm_M2")
     )
     (path "/4fec8b65-dfb4-433d-aad5-e8c79f736e6e"
-      (reference "H3") (unit 1) (value "MountingHole") (footprint "MountingHole:MountingHole_3.7mm")
+      (reference "H3") (unit 1) (value "MountingHole") (footprint "MountingHole:MountingHole_2.2mm_M2")
     )
     (path "/b8da359e-6266-4d68-9b60-2288812e8fe8"
-      (reference "H4") (unit 1) (value "MountingHole") (footprint "MountingHole:MountingHole_3.7mm")
+      (reference "H4") (unit 1) (value "MountingHole") (footprint "MountingHole:MountingHole_2.2mm_M2")
     )
     (path "/6e56e431-2312-4b78-ac6c-f2c9764450a6"
-      (reference "H5") (unit 1) (value "MountingHole") (footprint "MountingHole:MountingHole_3.7mm")
+      (reference "H5") (unit 1) (value "MountingHole") (footprint "MountingHole:MountingHole_2.2mm_M2")
     )
     (path "/e731a3eb-67ef-4303-aebd-6e657f2cbdf1"
-      (reference "H6") (unit 1) (value "MountingHole") (footprint "MountingHole:MountingHole_3.7mm")
+      (reference "H6") (unit 1) (value "MountingHole") (footprint "MountingHole:MountingHole_2.2mm_M2")
     )
     (path "/1e8f9367-136f-4c7d-8b2d-2f7dbe3d212b"
-      (reference "H7") (unit 1) (value "MountingHole") (footprint "MountingHole:MountingHole_3.7mm")
+      (reference "H7") (unit 1) (value "MountingHole") (footprint "MountingHole:MountingHole_2.2mm_M2")
     )
     (path "/090876d8-b41f-417b-b746-cba62def1acc"
-      (reference "H8") (unit 1) (value "MountingHole") (footprint "MountingHole:MountingHole_3.7mm")
+      (reference "H8") (unit 1) (value "MountingHole") (footprint "MountingHole:MountingHole_2.2mm_M2")
     )
   )
