File: SweepChoc/_MainPCB/sweepv2.kicad_sch (KiCad schematic)
At the start: 54 parts, among them J1 AudioJack4dpb, J2 AudioJack4dpb, SW1 SW_Push, SW10 SW_Push, SW11 SW_Push, SW11_r1 SW_Push, SW12 SW_Push, SW12_r1 SW_Push, SW13_r1 SW_Push, SW14 SW_Push, SW15 SW_Push, SW15_r1 SW_Push, SW16 SW_Push, SW16_r1 SW_Push, SW17 SW_Push, SW17_r1 SW_Push, SW18 SW_Push, SW18_r1 SW_Push, SW2 SW_Push, SW20 SW_Push, SW21 SW_Push, SW2_r1 SW_Push, SW3 SW_Push, SW3_r1 SW_Push, SW4 SW_Push, SW4_r1 SW_Push, SW5 SW_Push, SW5_r1 SW_Push, SW6 SW_Push, SW6_r1 SW_Push, SW7 SW_Push, SW7_r1 SW_Push, SW8 SW_Push, SW8_r1 SW_Push, SW9 SW_Push, SW9_r1 SW_Push, U1 ProMicro-kbd, U2 ProMicro-kbd

Commit message: re-worked choc version
Parts:
- RSW1, RSW2: value SW_Push -> Reset Button
- renumbered SW9_r1 to SW10_r1, SW7 to SW11_r1, SW11_r1 to SW12_r1, SW12_r1 to SW14_r1, SW13_r1 to SW15_r1, SW1 to SW16_r1, SW15_r1 to SW17_r1, SW16_r1 to SW18_r1, SW17_r1 to SW20_r1, SW18_r1 to SW21_r1, SW7_r1 to SW8_r1, SW8_r1 to SW9_r1
Connections:
- net raw: no longer SW_POWERR1.3 (C), U2.24 (RAW)
- net vcc: no longer J2.R1, U2.21 (VCC)
- new net raw_r: SW_POWERR1.3 (C), U2.24 (RAW)
- new net vcc_r: J2.R1, U2.21 (VCC)
